Commit message: Redefine object colors & set up first joint

File: src/inchworm/maria_inchworm_description/urdf/inchworm.urdf.xacro (robot description, xacro)
@@ -8,9 +8,23 @@
     </gazebo>
     <!-- Links -->
-    <link name="link1">
+    <link name="backfoot_link">
         <visual>
             <origin xyz="0 0 0" rpy="0 0 0"/>
             <geometry>
-                <mesh filename="package://maria_inchworm_description/meshes/InchwormFoot.obj"/>
+                <mesh filename="package://maria_inchworm_description/meshes/inchworm_foot.obj"/>
+            </geometry>
+        </visual>
+    </link>
+    <joint name="back_foot_leg_joint" type="continuous">
+        <origin xyz="0.0 0.0 0.0489" rpy="0.0 0.0 0.0"/>
+        <parent link="backfoot_link"/>
+        <child link="backleg_link"/>
+        <axis xyz="0 0 1"/>
+    </joint>
+    <link name="backleg_link">
+        <visual>
+            <origin xyz="0 0 0" rpy="0 0 0"/>
+            <geometry>
+                <mesh filename="package://maria_inchworm_description/meshes/inchworm_leg.obj"/>
             </geometry>
         </visual>

Commit message: Make xacro of inchworm, not considering dh params

File: src/inchworm/maria_inchworm_description/urdf/inchworm.urdf.xacro (robot description, xacro)
@@ -30,3 +30,59 @@
         </visual>
     </link>
+    <joint name="back_leg_c_link_joint" type="continuous">
+        <origin xyz="0.0 0.0 0.0573" rpy="-1.5707 2.7925 -3.1416"/>
+        <parent link="backleg_link"/>
+        <child link="c_link"/>
+        <axis xyz="0 0 1"/>
+    </joint>
+    <link name="c_link">
+        <visual>
+            <origin xyz="0 0 0.045" rpy="0 0 0"/>
+            <geometry>
+                <mesh filename="package://maria_inchworm_description/meshes/inchworm_clink.obj"/>
+            </geometry>
+        </visual>
+    </link>
+    <joint name="b_c_link_joint" type="continuous">
+        <origin xyz="0.0 0.1633 0.0" rpy="0 0 -2.4434"/>
+        <parent link="c_link"/>
+        <child link="b_link"/>
+        <axis xyz="0 0 1"/>
+    </joint>
+    <link name="b_link">
+        <visual>
+            <origin xyz="0 0 0.045" rpy="0 0 0"/>
+            <geometry>
+                <mesh filename="package://maria_inchworm_description/meshes/inchworm_blink.obj"/>
+            </geometry>
+        </visual>
+    </link>
+    <joint name="b_front_leg_joint" type="continuous">
+        <origin xyz="0.0 0.1633 0.0" rpy="0 0 -0.3491"/>
+        <parent link="b_link"/>
+        <child link="front_leg_link"/>
+        <axis xyz="0 0 1"/>
+    </joint>
+    <link name="front_leg_link">
+        <visual>
+            <origin xyz="0.0 0.0573 0" rpy="1.5707 3.14159 0"/>
+            <geometry>
+                <mesh filename="package://maria_inchworm_description/meshes/inchworm_leg.obj"/>
+            </geometry>
+        </visual>
+    </link>
+    <joint name="front_leg_foot_joint" type="continuous">
+        <origin xyz="0.0 0.0573 0.0" rpy="1.5707 0 0"/>
+        <parent link="front_leg_link"/>
+        <child link="front_foot_link"/>
+        <axis xyz="0 0 1"/>
+    </joint>
+    <link name="front_foot_link">
+        <visual>
+            <origin xyz="0.0 0 -0.0489" rpy="0 0 0"/>
+            <geometry>
+                <mesh filename="package://maria_inchworm_description/meshes/inchworm_foot.obj"/>
+            </geometry>
+        </visual>
+    </link>
 </robot>

Commit message: Modify inchworm xacro to follow dh parameters

File: src/inchworm/maria_inchworm_description/urdf/inchworm.urdf.xacro (robot description, xacro)
@@ -8,5 +8,91 @@
     </gazebo>
     <!-- Links -->
+    <link name="inchworm_main"/>
+    <link name="b_link">
+        <visual>
+            <origin xyz="0 0 0" rpy="0 0 0"/>
+            <geometry>
+                <mesh filename="package://maria_inchworm_description/meshes/inchworm_blink.obj"/>
+            </geometry>
+        </visual>
+    </link>
+    <link name="frontleg_link">
+        <visual>
+            <origin xyz="0 0 0" rpy="0 0 3.1416"/>
+            <geometry>
+                <mesh filename="package://maria_inchworm_description/meshes/inchworm_leg.obj"/>
+            </geometry>
+        </visual>
+    </link>
+    <link name="frontfoot_link">
+        <visual>
+            <origin xyz="0 0 0" rpy="0 0 0"/>
+            <geometry>
+                <mesh filename="package://maria_inchworm_description/meshes/inchworm_foot.obj"/>
+            </geometry>
+        </visual>
+    </link>
+    <link name="c_link">
+        <visual>
+            <origin xyz="0 0 0" rpy="0 0 0"/>
+            <geometry>
+                <mesh filename="package://maria_inchworm_description/meshes/inchworm_clink.obj"/>
+            </geometry>
+        </visual>
+    </link>
+    <link name="backleg_link">
+        <visual>
+            <origin xyz="0 0 0" rpy="0 0 3.1416"/>
+            <geometry>
+                <mesh filename="package://maria_inchworm_description/meshes/inchworm_leg.obj"/>
+            </geometry>
+        </visual>
+    </link>
     <link name="backfoot_link">
+        <visual>
+            <origin xyz="0 0 0" rpy="0 0 0"/>
+            <geometry>
+                <mesh filename="package://maria_inchworm_description/meshes/inchworm_foot.obj"/>
+            </geometry>
+        </visual>
+    </link>
+    <!-- Joints -->
+    <joint name="main_b_joint" type="continuous">
+        <origin xyz="0.0 0.0 0.0" rpy="-1.5707 0 0"/>
+        <parent link="inchworm_main"/>
+        <child link="b_link"/>
+        <axis xyz="0 0 1"/>
+    </joint>
+    <joint name="b_frontleg_joint" type="continuous">
+        <origin xyz="0.1633 0.0 0.0" rpy="0 0 0"/>
+        <parent link="b_link"/>
+        <child link="frontleg_link"/>
+        <axis xyz="0 0 1"/>
+    </joint>
+    <joint name="frontleg_frontfoot_joint" type="continuous">
+        <origin xyz="0.0573 0.0 0.0" rpy="1.5707 0.0 -1.5707"/>
+        <parent link="frontleg_link"/>
+        <child link="frontfoot_link"/>
+        <axis xyz="0 0 1"/>
+    </joint>
+    <joint name="main_c_joint" type="continuous">
+        <origin xyz="0.0 0.0 0.0" rpy="-1.5707 3.1416 0"/>
+        <parent link="inchworm_main"/>
+        <child link="c_link"/>
+        <axis xyz="0 0 1"/>
+    </joint>
+    <joint name="c_backleg_joint" type="continuous">
+        <origin xyz="0.1633 0.0 0.0" rpy="0 0 0"/>
+        <parent link="c_link"/>
+        <child link="backleg_link"/>
+        <axis xyz="0 0 1"/>
+    </joint>
+    <joint name="backleg_backfoot_joint" type="continuous">
+        <origin xyz="0.0573 0.0 0.0" rpy="1.5707 0.0 -1.5707"/>
+        <parent link="backleg_link"/>
+        <child link="backfoot_link"/>
+        <axis xyz="0 0 1"/>
+    </joint>
+    <!-- <link name="backfoot_link">
         <visual>
             <origin xyz="0 0 0" rpy="0 0 0"/>
@@ -86,3 +172,4 @@
         </visual>
     </link>
+     -->
 </robot>
