Commit message: Add working playground but non-working robot

File: src/inchworm_project_gazebo/urdf/playground.urdf.xacro (robot description, xacro)
@@ -14,10 +14,5 @@
         <origin xyz="0.0 0.0 0.0" rpy="0.0 0.0 0.0"/>
         <parent link="world"/>
-        <!-- Uncomment below if you want to test general kinematics or end effector -->
         <child link="playground"/>
-        <!-- Uncomment below if you want to test front foot kinematics -->
-        <!-- <child link="backfoot_ee_link"/>  -->
-        <!-- Uncomment below if you want to test back foot kinematics -->
-        <!-- <child link="frontfoot_link"/>  -->
     </joint>
     <!-- Links -->
@@ -26,5 +21,5 @@
             <origin xyz="0 0 0" rpy="0 0 0"/>
             <geometry>
-                <mesh filename="package://inchworm_project_gazebo/models/playground/playground.dae"/>
+                <mesh filename="package://inchworm_project_gazebo/meshes/playground.dae"/>
             </geometry>
         </visual>
@@ -32,5 +27,5 @@
             <origin xyz="0 0 0" rpy="0.0 0.0 0.0"/>
             <geometry>
-                <mesh filename="package://inchworm_project_gazebo/models/playground/playground.dae"/>
+                <mesh filename="package://inchworm_project_gazebo/meshes/playground.dae"/>
             </geometry>
         </collision>

Commit message: Add working static inchworm environment

File: src/inchworm_project_gazebo/urdf/playground.urdf.xacro (robot description, xacro)
@@ -4,12 +4,7 @@
     The inchworm will be fixed to a specific position as determined under 'Static Joint to World Frame' comment -->
     <!-- Import Gazebo ROS Control Plugin -->
-    <gazebo>
-        <plugin name="gazebo_ros_control" filename="libgazebo_ros_control.so">
-            <robotNamespace>/playground</robotNamespace>
-        </plugin>
-    </gazebo>
     <!-- Static Joint to World Frame in Simulation -->
     <link name="world"/>
-    <joint name="joint_name" type="fixed">
+    <joint name="world_playground_joint" type="fixed">
         <origin xyz="0.0 0.0 0.0" rpy="0.0 0.0 0.0"/>
         <parent link="world"/>

Commit message: Add modified launch file to include init_config script

File: src/inchworm_project_gazebo/urdf/playground.urdf.xacro (robot description, xacro)
@@ -27,5 +27,5 @@
         <inertial>
             <origin xyz="0.0 0.0 0.0" rpy="0.0 0.0 0.0"/>
-            <mass value="0.1"/>
+            <mass value="1000.0"/>
             <inertia ixx="0.0" ixy="0.0" ixz="0.0" iyy="0.0" iyz="0.0" izz="0.0"/>
         </inertial>
