Commit message: Fix gazebo display and crashing issues

File: src/inchworm/inchworm_description/urdf/inchworm_static.urdf.xacro (robot description, xacro)
@@ -22,15 +22,21 @@
     </joint>
     <!-- Links -->
-    <link name="inchworm_main"/>
+    <link name="inchworm_main">
+        <inertial>
+            <origin xyz="0.0 0.0 0.0" rpy="0.0 0.0 0.0"/>
+            <mass value="0.001"/>
+            <inertia ixx="0.0" ixy="0.0" ixz="0.0" iyy="0.0" iyz="0.0" izz="0.0"/>
+        </inertial>
+    </link>
     <link name="b_link">
         <visual>
             <origin xyz="0 0 0" rpy="0 0 0"/>
             <geometry>
-                <mesh filename="package://inchworm_description/meshes/inchworm_blink.obj"/>
+                <mesh filename="package://inchworm_description/meshes/inchworm_blink.dae"/>
             </geometry>
         </visual>
         <inertial>
             <origin xyz="0.0 0.0 0.0" rpy="0.0 0.0 0.0"/>
-            <mass value="0.0"/>
+            <mass value="0.1"/>
             <inertia ixx="0.0" ixy="0.0" ixz="0.0" iyy="0.0" iyz="0.0" izz="0.0"/>
         </inertial>
@@ -40,10 +46,10 @@
             <origin xyz="0 0 0" rpy="0 0 3.1416"/>
             <geometry>
-                <mesh filename="package://inchworm_description/meshes/inchworm_leg.obj"/>
+                <mesh filename="package://inchworm_description/meshes/inchworm_leg.dae"/>
             </geometry>
         </visual>
         <inertial>
             <origin xyz="0.0 0.0 0.0" rpy="0.0 0.0 0.0"/>
-            <mass value="0.0"/>
+            <mass value="0.1"/>
             <inertia ixx="0.0" ixy="0.0" ixz="0.0" iyy="0.0" iyz="0.0" izz="0.0"/>
         </inertial>
@@ -53,14 +59,19 @@
             <origin xyz="0 0 0" rpy="0 0 0"/>
             <geometry>
-                <mesh filename="package://inchworm_description/meshes/inchworm_foot.obj"/>
+                <mesh filename="package://inchworm_description/meshes/inchworm_foot.dae"/>
             </geometry>
         </visual>
         <inertial>
             <origin xyz="0.0 0.0 0.0" rpy="0.0 0.0 0.0"/>
-            <mass value="0.0"/>
+            <mass value="0.1"/>
             <inertia ixx="0.0" ixy="0.0" ixz="0.0" iyy="0.0" iyz="0.0" izz="0.0"/>
         </inertial>
     </link>
     <link name="frontfoot_ee_link">
+        <inertial>
+            <origin xyz="0.0 0.0 0.0" rpy="0.0 0.0 0.0"/>
+            <mass value="0.1"/>
+            <inertia ixx="0.0" ixy="0.0" ixz="0.0" iyy="0.0" iyz="0.0" izz="0.0"/>
+        </inertial>
     </link>
     <link name="c_link">
@@ -68,10 +79,10 @@
             <origin xyz="0 0 0" rpy="0 0 0"/>
             <geometry>
-                <mesh filename="package://inchworm_description/meshes/inchworm_clink.obj"/>
+                <mesh filename="package://inchworm_description/meshes/inchworm_clink.dae"/>
             </geometry>
         </visual>
         <inertial>
             <origin xyz="0.0 0.0 0.0" rpy="0.0 0.0 0.0"/>
-            <mass value="0.0"/>
+            <mass value="0.1"/>
             <inertia ixx="0.0" ixy="0.0" ixz="0.0" iyy="0.0" iyz="0.0" izz="0.0"/>
         </inertial>
@@ -81,10 +92,10 @@
             <origin xyz="0 0 0" rpy="0 0 3.1416"/>
             <geometry>
-                <mesh filename="package://inchworm_description/meshes/inchworm_leg.obj"/>
+                <mesh filename="package://inchworm_description/meshes/inchworm_leg.dae"/>
             </geometry>
         </visual>
         <inertial>
             <origin xyz="0.0 0.0 0.0" rpy="0.0 0.0 0.0"/>
-            <mass value="0.0"/>
+            <mass value="0.1"/>
             <inertia ixx="0.0" ixy="0.0" ixz="0.0" iyy="0.0" iyz="0.0" izz="0.0"/>
         </inertial>
@@ -94,14 +105,19 @@
             <origin xyz="0 0 0" rpy="0 0 0"/>
             <geometry>
-                <mesh filename="package://inchworm_description/meshes/inchworm_foot.obj"/>
+                <mesh filename="package://inchworm_description/meshes/inchworm_foot.dae"/>
             </geometry>
         </visual>
         <inertial>
             <origin xyz="0.0 0.0 0.0" rpy="0.0 0.0 0.0"/>
-            <mass value="0.0"/>
+            <mass value="0.1"/>
             <inertia ixx="0.0" ixy="0.0" ixz="0.0" iyy="0.0" iyz="0.0" izz="0.0"/>
         </inertial>
     </link>
     <link name="backfoot_ee_link">
+        <inertial>
+            <origin xyz="0.0 0.0 0.0" rpy="0.0 0.0 0.0"/>
+            <mass value="0.1"/>
+            <inertia ixx="0.0" ixy="0.0" ixz="0.0" iyy="0.0" iyz="0.0" izz="0.0"/>
+        </inertial>
     </link>
     <!-- Joints -->

Commit message: Add transmission interface to the static urdf model

File: src/inchworm/inchworm_description/urdf/inchworm_static.urdf.xacro (robot description, xacro)
@@ -121,4 +121,14 @@
         </inertial>
     </link>
+    <!-- Joint Transmission Macro -->
+    <xacro:macro name="joint_transmission" params="prefix">
+        <transmission name="${prefix}_transmission">
+            <type>transmission_interface/SimpleTransmission</type>
+            <joint name="${prefix}_joint">
+                <hardwareInterface>hardware_interface/PositionJointInterface</hardwareInterface>
+            </joint>
+            <actuator name="${prefix}_motor"></actuator>
+        </transmission>
+    </xacro:macro>
     <!-- Joints -->
     <joint name="main_b_joint" type="continuous">
@@ -128,4 +138,5 @@
         <axis xyz="0 0 1"/>
     </joint>
+    <xacro:joint_transmission prefix="main_b"/>
     <joint name="b_frontleg_joint" type="continuous">
         <origin xyz="0.1633 0.0 0.0" rpy="0 0 0"/>
@@ -134,4 +145,5 @@
         <axis xyz="0 0 1"/>
     </joint>
+    <xacro:joint_transmission prefix="b_frontleg"/>
     <joint name="frontleg_frontfoot_joint" type="continuous">
         <origin xyz="0.0573 0.0 0.0" rpy="1.5707 0.0 -1.5707"/>
@@ -140,4 +152,5 @@
         <axis xyz="0 0 1"/>
     </joint>
+    <xacro:joint_transmission prefix="frontleg_frontfoot"/>
     <joint name="frontfoot_ee_joint" type="fixed">
         <origin xyz="0.0 0.0 -0.0489" rpy="0.0 0.0 0.0"/>
@@ -151,4 +164,5 @@
         <axis xyz="0 0 1"/>
     </joint>
+    <xacro:joint_transmission prefix="main_c"/>
     <joint name="c_backleg_joint" type="continuous">
         <origin xyz="0.1633 0.0 0.0" rpy="0 0 0"/>
@@ -157,4 +171,5 @@
         <axis xyz="0 0 1"/>
     </joint>
+    <xacro:joint_transmission prefix="c_backleg"/>
     <joint name="backleg_backfoot_joint" type="continuous">
         <origin xyz="0.0573 0.0 0.0" rpy="1.5707 0.0 -1.5707"/>
@@ -163,4 +178,5 @@
         <axis xyz="0 0 1"/>
     </joint>
+    <xacro:joint_transmission prefix="backleg_backfoot"/>
     <joint name="backfoot_ee_joint" type="fixed">
         <origin xyz="0.0 0.0 -0.0489" rpy="0.0 0.0 0.0"/>

Commit message: Add proposal paper final and some changes to the urdf

File: src/inchworm/inchworm_description/urdf/inchworm_static.urdf.xacro (robot description, xacro)
@@ -9,4 +9,7 @@
         </plugin>
     </gazebo>
+    <!-- Joint Properties -->
+    <xacro:property name="joint_speed" value="545"/>        <!-- in rpm -->
+    <xacro:property name="joint_torque" value="0.03525"/>   <!-- in N-m -->
     <!-- Static Joint to World Frame in Simulation -->
     <link name="world"/>
@@ -137,4 +140,6 @@
         <child link="b_link"/>
         <axis xyz="0 0 1"/>
+        <limit  effort="${joint_torque}"
+                velocity="${joint_speed * 2 * 3.14159 / 60 }"/>
     </joint>
     <xacro:joint_transmission prefix="main_b"/>
@@ -144,4 +149,6 @@
         <child link="frontleg_link"/>
         <axis xyz="0 0 1"/>
+        <limit  effort="${joint_torque}"
+                velocity="${joint_speed * 2 * 3.14159 / 60 }"/>
     </joint>
     <xacro:joint_transmission prefix="b_frontleg"/>
@@ -151,4 +158,6 @@
         <child link="frontfoot_link"/>
         <axis xyz="0 0 1"/>
+        <limit  effort="${joint_torque}"
+                velocity="${joint_speed * 2 * 3.14159 / 60 }"/>
     </joint>
     <xacro:joint_transmission prefix="frontleg_frontfoot"/>
@@ -157,4 +166,6 @@
         <parent link="frontfoot_link"/>
         <child link="frontfoot_ee_link"/>
+        <limit  effort="${joint_torque}"
+                velocity="${joint_speed * 2 * 3.14159 / 60 }"/>
     </joint>
     <joint name="main_c_joint" type="continuous">
@@ -163,4 +174,6 @@
         <child link="c_link"/>
         <axis xyz="0 0 1"/>
+        <limit  effort="${joint_torque}"
+                velocity="${joint_speed * 2 * 3.14159 / 60 }"/>
     </joint>
     <xacro:joint_transmission prefix="main_c"/>
@@ -170,4 +183,6 @@
         <child link="backleg_link"/>
         <axis xyz="0 0 1"/>
+        <limit  effort="${joint_torque}"
+                velocity="${joint_speed * 2 * 3.14159 / 60 }"/>
     </joint>
     <xacro:joint_transmission prefix="c_backleg"/>
@@ -177,4 +192,6 @@
         <child link="backfoot_link"/>
         <axis xyz="0 0 1"/>
+        <limit  effort="${joint_torque}"
+                velocity="${joint_speed * 2 * 3.14159 / 60 }"/>
     </joint>
     <xacro:joint_transmission prefix="backleg_backfoot"/>
@@ -183,4 +200,6 @@
         <parent link="backfoot_link"/>
         <child link="backfoot_ee_link"/>
+        <limit  effort="${joint_torque}"
+                velocity="${joint_speed * 2 * 3.14159 / 60 }"/>
     </joint>
 </robot>

Commit message: Add non-working playground files

File: src/inchworm/inchworm_description/urdf/inchworm_static.urdf.xacro (robot description, xacro)
@@ -20,5 +20,5 @@
         <child link="inchworm_main"/>
         <!-- Uncomment below if you want to test front foot kinematics -->
-        <!-- <child link="backfoot_link"/>  -->
+        <!-- <child link="backfoot_ee_link"/>  -->
         <!-- Uncomment below if you want to test back foot kinematics -->
         <!-- <child link="frontfoot_link"/>  -->

Commit message: Adding in inertia vales for all links

File: src/inchworm/inchworm_description/urdf/inchworm_static.urdf.xacro (robot description, xacro)
@@ -1,3 +1,3 @@
-<?xml version="1.0"?>
+ <?xml version="1.0"?>
 <robot xmlns:xacro="http://wiki.ros.org/xacro" name="inchworm_static">
     <!-- Note: Only use this URDF when testing the inchworm kinematics.
@@ -41,9 +41,55 @@
         <inertial>
             <origin xyz="0.0 0.0 0.0" rpy="0.0 0.0 0.0"/>
+            <mass value="0.0997"/>
+            <inertia ixx="182.79" ixy="0.0" ixz="-35.15" iyy="2572.23" iyz="0.0" izz="2446.68"/>
+        </inertial>
+    </link>
+    <link name="frontleg_link">
+        <visual>
+            <origin xyz="0 0 0" rpy="0 0 3.1416"/>
+            <geometry>
+                <mesh filename="package://inchworm_description/meshes/inchworm_leg.dae"/>
+            </geometry>
+        </visual>
+        <inertial>
+            <origin xyz="0.0 0.0 0.0" rpy="0.0 0.0 0.0"/>
+            <mass value="0.0181"/>
+            <inertia ixx="056.24" ixy="0.0" ixz="-21.09" iyy="84.36" iyz="0.0" izz="14.06"/>
+        </inertial>
+    </link>
+    <link name="frontfoot_link">
+        <visual>
+            <origin xyz="0 0 0" rpy="0 0 0"/>
+            <geometry>
+                <mesh filename="package://inchworm_description/meshes/inchworm_foot.dae"/>
+            </geometry>
+        </visual>
+        <inertial>
+            <origin xyz="0.0 0.0 0.0" rpy="0.0 0.0 0.0"/>
+            <mass value="0.09525"/>
+            <inertia ixx="358.56" ixy="0.0" ixz="0.0" iyy="337.47" iyz="0.0" izz="98.47"/>
+        </inertial>
+    </link>
+    <link name="frontfoot_ee_link">
+        <inertial>
+            <origin xyz="0.0 0.0 0.0" rpy="0.0 0.0 0.0"/>
             <mass value="0.1"/>
             <inertia ixx="0.0" ixy="0.0" ixz="0.0" iyy="0.0" iyz="0.0" izz="0.0"/>
         </inertial>
     </link>
-    <link name="frontleg_link">
+    <link name="c_link">
+        <visual>
+            <origin xyz="0 0 0" rpy="0 0 0"/>
+            <geometry>
+                <mesh filename="package://inchworm_description/meshes/inchworm_clink.dae"/>
+            </geometry>
+        </visual>
+        <inertial>
+            <origin xyz="0.0 0.0 0.0" rpy="0.0 0.0 0.0"/>
+            <mass value="0.1995"/>
+            <inertia ixx="379.65" ixy="-21.95" ixz="435.90" iyy="5673.77" iyz="-28.12" izz="1195.21"/>
+        </inertial>
+    </link>
+    <link name="backleg_link">
         <visual>
             <origin xyz="0 0 0" rpy="0 0 3.1416"/>
@@ -54,9 +100,9 @@
         <inertial>
             <origin xyz="0.0 0.0 0.0" rpy="0.0 0.0 0.0"/>
-            <mass value="0.1"/>
-            <inertia ixx="0.0" ixy="0.0" ixz="0.0" iyy="0.0" iyz="0.0" izz="0.0"/>
-        </inertial>
-    </link>
-    <link name="frontfoot_link">
+            <mass value="0.09525"/>
+            <inertia ixx="358.56" ixy="0.0" ixz="0.0" iyy="337.47" iyz="0.0" izz="98.47"/>
+        </inertial>
+    </link>
+    <link name="backfoot_link">
         <visual>
             <origin xyz="0 0 0" rpy="0 0 0"/>
@@ -67,52 +113,6 @@
         <inertial>
             <origin xyz="0.0 0.0 0.0" rpy="0.0 0.0 0.0"/>
-            <mass value="0.1"/>
-            <inertia ixx="0.0" ixy="0.0" ixz="0.0" iyy="0.0" iyz="0.0" izz="0.0"/>
-        </inertial>
-    </link>
-    <link name="frontfoot_ee_link">
-        <inertial>
-            <origin xyz="0.0 0.0 0.0" rpy="0.0 0.0 0.0"/>
-            <mass value="0.1"/>
-            <inertia ixx="0.0" ixy="0.0" ixz="0.0" iyy="0.0" iyz="0.0" izz="0.0"/>
-        </inertial>
-    </link>
-    <link name="c_link">
-        <visual>
-            <origin xyz="0 0 0" rpy="0 0 0"/>
-            <geometry>
-                <mesh filename="package://inchworm_description/meshes/inchworm_clink.dae"/>
-            </geometry>
-        </visual>
-        <inertial>
-            <origin xyz="0.0 0.0 0.0" rpy="0.0 0.0 0.0"/>
-            <mass value="0.1"/>
-            <inertia ixx="0.0" ixy="0.0" ixz="0.0" iyy="0.0" iyz="0.0" izz="0.0"/>
-        </inertial>
-    </link>
-    <link name="backleg_link">
-        <visual>
-            <origin xyz="0 0 0" rpy="0 0 3.1416"/>
-            <geometry>
-                <mesh filename="package://inchworm_description/meshes/inchworm_leg.dae"/>
-            </geometry>
-        </visual>
-        <inertial>
-            <origin xyz="0.0 0.0 0.0" rpy="0.0 0.0 0.0"/>
-            <mass value="0.1"/>
-            <inertia ixx="0.0" ixy="0.0" ixz="0.0" iyy="0.0" iyz="0.0" izz="0.0"/>
-        </inertial>
-    </link>
-    <link name="backfoot_link">
-        <visual>
-            <origin xyz="0 0 0" rpy="0 0 0"/>
-            <geometry>
-                <mesh filename="package://inchworm_description/meshes/inchworm_foot.dae"/>
-            </geometry>
-        </visual>
-        <inertial>
-            <origin xyz="0.0 0.0 0.0" rpy="0.0 0.0 0.0"/>
-            <mass value="0.1"/>
-            <inertia ixx="0.0" ixy="0.0" ixz="0.0" iyy="0.0" iyz="0.0" izz="0.0"/>
+            <mass value="0.09525"/>
+            <inertia ixx="358.56" ixy="0.0" ixz="0.0" iyy="337.47" iyz="0.0" izz="98.47"/>
         </inertial>
     </link>
