Commit message: Add end effector links to the URDF

File: src/inchworm/inchworm_description/urdf/inchworm.urdf.xacro (robot description, xacro)
@@ -33,4 +33,6 @@
         </visual>
     </link>
+    <link name="frontfoot_ee_link">
+    </link>
     <link name="c_link">
         <visual>
@@ -57,4 +59,6 @@
         </visual>
     </link>
+    <link name="backfoot_ee_link">
+    </link>
     <!-- Joints -->
     <joint name="main_b_joint" type="continuous">
@@ -76,4 +80,9 @@
         <axis xyz="0 0 1"/>
     </joint>
+    <joint name="frontfoot_ee_joint" type="fixed">
+        <origin xyz="0.0 0.0 -0.0489" rpy="0.0 0.0 0.0"/>
+        <parent link="frontfoot_link"/>
+        <child link="frontfoot_ee_link"/>
+    </joint>
     <joint name="main_c_joint" type="continuous">
         <origin xyz="0.0 0.0 0.0" rpy="-1.5707 3.1416 0"/>
@@ -94,3 +103,8 @@
         <axis xyz="0 0 1"/>
     </joint>
+    <joint name="backfoot_ee_joint" type="fixed">
+        <origin xyz="0.0 0.0 -0.0489" rpy="0.0 0.0 0.0"/>
+        <parent link="backfoot_link"/>
+        <child link="backfoot_ee_link"/>
+    </joint>
 </robot>

Commit message: add interface to control joints in the inchworm class

File: src/inchworm/inchworm_description/urdf/inchworm.urdf.xacro (robot description, xacro)
@@ -8,12 +8,23 @@
     </gazebo>
     <!-- Links -->
-    <link name="inchworm_main"/>
+    <link name="inchworm_main">
+        <inertial>
+            <origin xyz="0.0 0.0 0.0" rpy="0.0 0.0 0.0"/>
+            <mass value="0.001"/>
+            <inertia ixx="0.0" ixy="0.0" ixz="0.0" iyy="0.0" iyz="0.0" izz="0.0"/>
+        </inertial>
+    </link>
     <link name="b_link">
         <visual>
             <origin xyz="0 0 0" rpy="0 0 0"/>
             <geometry>
-                <mesh filename="package://inchworm_description/meshes/inchworm_blink.obj"/>
+                <mesh filename="package://inchworm_description/meshes/inchworm_blink.dae"/>
             </geometry>
         </visual>
+        <inertial>
+            <origin xyz="0.0 0.0 0.0" rpy="0.0 0.0 0.0"/>
+            <mass value="0.1"/>
+            <inertia ixx="0.0" ixy="0.0" ixz="0.0" iyy="0.0" iyz="0.0" izz="0.0"/>
+        </inertial>
     </link>
     <link name="frontleg_link">
@@ -21,7 +32,12 @@
             <origin xyz="0 0 0" rpy="0 0 3.1416"/>
             <geometry>
-                <mesh filename="package://inchworm_description/meshes/inchworm_leg.obj"/>
+                <mesh filename="package://inchworm_description/meshes/inchworm_leg.dae"/>
             </geometry>
         </visual>
+        <inertial>
+            <origin xyz="0.0 0.0 0.0" rpy="0.0 0.0 0.0"/>
+            <mass value="0.1"/>
+            <inertia ixx="0.0" ixy="0.0" ixz="0.0" iyy="0.0" iyz="0.0" izz="0.0"/>
+        </inertial>
     </link>
     <link name="frontfoot_link">
@@ -29,9 +45,19 @@
             <origin xyz="0 0 0" rpy="0 0 0"/>
             <geometry>
-                <mesh filename="package://inchworm_description/meshes/inchworm_foot.obj"/>
+                <mesh filename="package://inchworm_description/meshes/inchworm_foot.dae"/>
             </geometry>
         </visual>
+        <inertial>
+            <origin xyz="0.0 0.0 0.0" rpy="0.0 0.0 0.0"/>
+            <mass value="0.1"/>
+            <inertia ixx="0.0" ixy="0.0" ixz="0.0" iyy="0.0" iyz="0.0" izz="0.0"/>
+        </inertial>
     </link>
     <link name="frontfoot_ee_link">
+        <inertial>
+            <origin xyz="0.0 0.0 0.0" rpy="0.0 0.0 0.0"/>
+            <mass value="0.1"/>
+            <inertia ixx="0.0" ixy="0.0" ixz="0.0" iyy="0.0" iyz="0.0" izz="0.0"/>
+        </inertial>
     </link>
     <link name="c_link">
@@ -39,7 +65,12 @@
             <origin xyz="0 0 0" rpy="0 0 0"/>
             <geometry>
-                <mesh filename="package://inchworm_description/meshes/inchworm_clink.obj"/>
+                <mesh filename="package://inchworm_description/meshes/inchworm_clink.dae"/>
             </geometry>
         </visual>
+        <inertial>
+            <origin xyz="0.0 0.0 0.0" rpy="0.0 0.0 0.0"/>
+            <mass value="0.1"/>
+            <inertia ixx="0.0" ixy="0.0" ixz="0.0" iyy="0.0" iyz="0.0" izz="0.0"/>
+        </inertial>
     </link>
     <link name="backleg_link">
@@ -47,7 +78,12 @@
             <origin xyz="0 0 0" rpy="0 0 3.1416"/>
             <geometry>
-                <mesh filename="package://inchworm_description/meshes/inchworm_leg.obj"/>
+                <mesh filename="package://inchworm_description/meshes/inchworm_leg.dae"/>
             </geometry>
         </visual>
+        <inertial>
+            <origin xyz="0.0 0.0 0.0" rpy="0.0 0.0 0.0"/>
+            <mass value="0.1"/>
+            <inertia ixx="0.0" ixy="0.0" ixz="0.0" iyy="0.0" iyz="0.0" izz="0.0"/>
+        </inertial>
     </link>
     <link name="backfoot_link">
@@ -55,17 +91,38 @@
             <origin xyz="0 0 0" rpy="0 0 0"/>
             <geometry>
-                <mesh filename="package://inchworm_description/meshes/inchworm_foot.obj"/>
+                <mesh filename="package://inchworm_description/meshes/inchworm_foot.dae"/>
             </geometry>
         </visual>
+        <inertial>
+            <origin xyz="0.0 0.0 0.0" rpy="0.0 0.0 0.0"/>
+            <mass value="0.1"/>
+            <inertia ixx="0.0" ixy="0.0" ixz="0.0" iyy="0.0" iyz="0.0" izz="0.0"/>
+        </inertial>
     </link>
     <link name="backfoot_ee_link">
+        <inertial>
+            <origin xyz="0.0 0.0 0.0" rpy="0.0 0.0 0.0"/>
+            <mass value="0.1"/>
+            <inertia ixx="0.0" ixy="0.0" ixz="0.0" iyy="0.0" iyz="0.0" izz="0.0"/>
+        </inertial>
     </link>
+    <!-- Joint Transmission Macro -->
+    <xacro:macro name="joint_transmission" params="prefix">
+        <transmission name="${prefix}_transmission">
+            <type>transmission_interface/SimpleTransmission</type>
+            <joint name="${prefix}_joint">
+                <hardwareInterface>hardware_interface/PositionJointInterface</hardwareInterface>
+            </joint>
+            <actuator name="${prefix}_motor"></actuator>
+        </transmission>
+    </xacro:macro>
     <!-- Joints -->
     <joint name="main_b_joint" type="continuous">
-        <origin xyz="0.0 0.0 0.0" rpy="-1.5707 0 0"/>
+        <origin xyz="0.0 0.0 0.0" rpy="-1.5707 1.5707 0"/>
         <parent link="inchworm_main"/>
         <child link="b_link"/>
         <axis xyz="0 0 1"/>
     </joint>
+    <xacro:joint_transmission prefix="main_b"/>
     <joint name="b_frontleg_joint" type="continuous">
         <origin xyz="0.1633 0.0 0.0" rpy="0 0 0"/>
@@ -74,4 +131,5 @@
         <axis xyz="0 0 1"/>
     </joint>
+    <xacro:joint_transmission prefix="b_frontleg"/>
     <joint name="frontleg_frontfoot_joint" type="continuous">
         <origin xyz="0.0573 0.0 0.0" rpy="1.5707 0.0 -1.5707"/>
@@ -80,4 +138,5 @@
         <axis xyz="0 0 1"/>
     </joint>
+    <xacro:joint_transmission prefix="frontleg_frontfoot"/>
     <joint name="frontfoot_ee_joint" type="fixed">
         <origin xyz="0.0 0.0 -0.0489" rpy="0.0 0.0 0.0"/>
@@ -86,9 +145,10 @@
     </joint>
     <joint name="main_c_joint" type="continuous">
-        <origin xyz="0.0 0.0 0.0" rpy="-1.5707 3.1416 0"/>
+        <origin xyz="0.0 0.0 0.0" rpy="-1.5707 1.5707 0"/>
         <parent link="inchworm_main"/>
         <child link="c_link"/>
         <axis xyz="0 0 1"/>
     </joint>
+    <xacro:joint_transmission prefix="main_c"/>
     <joint name="c_backleg_joint" type="continuous">
         <origin xyz="0.1633 0.0 0.0" rpy="0 0 0"/>
@@ -97,4 +157,5 @@
         <axis xyz="0 0 1"/>
     </joint>
+    <xacro:joint_transmission prefix="c_backleg"/>
     <joint name="backleg_backfoot_joint" type="continuous">
         <origin xyz="0.0573 0.0 0.0" rpy="1.5707 0.0 -1.5707"/>
@@ -103,4 +164,5 @@
         <axis xyz="0 0 1"/>
     </joint>
+    <xacro:joint_transmission prefix="backleg_backfoot"/>
     <joint name="backfoot_ee_joint" type="fixed">
         <origin xyz="0.0 0.0 -0.0489" rpy="0.0 0.0 0.0"/>

File: src/inchworm/inchworm_description/urdf/inchworm_static.urdf.xacro (robot description, xacro)
@@ -133,5 +133,5 @@
     <!-- Joints -->
     <joint name="main_b_joint" type="continuous">
-        <origin xyz="0.0 0.0 0.0" rpy="-1.5707 0 0"/>
+        <origin xyz="0.0 0.0 0.0" rpy="-1.5707 1.5707 0"/>
         <parent link="inchworm_main"/>
         <child link="b_link"/>
@@ -159,5 +159,5 @@
     </joint>
     <joint name="main_c_joint" type="continuous">
-        <origin xyz="0.0 0.0 0.0" rpy="-1.5707 3.1416 0"/>
+        <origin xyz="0.0 0.0 0.0" rpy="-1.5707 1.5707 0"/>
         <parent link="inchworm_main"/>
         <child link="c_link"/>

Commit message: Add non-working free urdf

File: src/inchworm/inchworm_description/urdf/inchworm.urdf.xacro (robot description, xacro)
@@ -1,4 +1,6 @@
 <?xml version="1.0"?>
 <robot xmlns:xacro="http://wiki.ros.org/xacro" name="inchworm">
+    <!-- Note: Only use this URDF when testing the inchworm kinematics.
+    The inchworm will be fixed to a specific position as determined under 'Static Joint to World Frame' comment -->
     <!-- Import Gazebo ROS Control Plugin -->
     <gazebo>
@@ -7,4 +9,14 @@
         </plugin>
     </gazebo>
+    <!-- Joint Properties -->
+    <xacro:property name="joint_speed" value="545"/>        <!-- in rpm -->
+    <xacro:property name="joint_torque" value="0.03525"/>   <!-- in N-m -->
+    <!-- Static Joint to World Frame in Simulation -->
+    <link name="world"/>
+    <joint name="joint_name" type="fixed">
+        <origin xyz="0.0 0.0 0.0" rpy="0.0 0.0 0.0"/>
+        <parent link="world"/>
+        <child link="inchworm_main"/>
+    </joint>
     <!-- Links -->
     <link name="inchworm_main">
@@ -123,4 +135,6 @@
         <child link="b_link"/>
         <axis xyz="0 0 1"/>
+        <limit  effort="${joint_torque}"
+                velocity="${joint_speed * 2 * 3.14159 / 60 }"/>
     </joint>
     <xacro:joint_transmission prefix="main_b"/>
@@ -130,4 +144,6 @@
         <child link="frontleg_link"/>
         <axis xyz="0 0 1"/>
+        <limit  effort="${joint_torque}"
+                velocity="${joint_speed * 2 * 3.14159 / 60 }"/>
     </joint>
     <xacro:joint_transmission prefix="b_frontleg"/>
@@ -137,4 +153,6 @@
         <child link="frontfoot_link"/>
         <axis xyz="0 0 1"/>
+        <limit  effort="${joint_torque}"
+                velocity="${joint_speed * 2 * 3.14159 / 60 }"/>
     </joint>
     <xacro:joint_transmission prefix="frontleg_frontfoot"/>
@@ -143,4 +161,6 @@
         <parent link="frontfoot_link"/>
         <child link="frontfoot_ee_link"/>
+        <limit  effort="${joint_torque}"
+                velocity="${joint_speed * 2 * 3.14159 / 60 }"/>
     </joint>
     <joint name="main_c_joint" type="continuous">
@@ -149,4 +169,6 @@
         <child link="c_link"/>
         <axis xyz="0 0 1"/>
+        <limit  effort="${joint_torque}"
+                velocity="${joint_speed * 2 * 3.14159 / 60 }"/>
     </joint>
     <xacro:joint_transmission prefix="main_c"/>
@@ -156,4 +178,6 @@
         <child link="backleg_link"/>
         <axis xyz="0 0 1"/>
+        <limit  effort="${joint_torque}"
+                velocity="${joint_speed * 2 * 3.14159 / 60 }"/>
     </joint>
     <xacro:joint_transmission prefix="c_backleg"/>
@@ -163,4 +187,6 @@
         <child link="backfoot_link"/>
         <axis xyz="0 0 1"/>
+        <limit  effort="${joint_torque}"
+                velocity="${joint_speed * 2 * 3.14159 / 60 }"/>
     </joint>
     <xacro:joint_transmission prefix="backleg_backfoot"/>
@@ -169,4 +195,6 @@
         <parent link="backfoot_link"/>
         <child link="backfoot_ee_link"/>
+        <limit  effort="${joint_torque}"
+                velocity="${joint_speed * 2 * 3.14159 / 60 }"/>
     </joint>
 </robot>

Commit message: Add working dynamic inchworm, no collision models

File: src/inchworm/inchworm_description/urdf/inchworm.urdf.xacro (robot description, xacro)
@@ -12,11 +12,4 @@
     <xacro:property name="joint_speed" value="545"/>        <!-- in rpm -->
     <xacro:property name="joint_torque" value="0.03525"/>   <!-- in N-m -->
-    <!-- Static Joint to World Frame in Simulation -->
-    <link name="world"/>
-    <joint name="joint_name" type="fixed">
-        <origin xyz="0.0 0.0 0.0" rpy="0.0 0.0 0.0"/>
-        <parent link="world"/>
-        <child link="inchworm_main"/>
-    </joint>
     <!-- Links -->
     <link name="inchworm_main">

Commit message: Add collision models to the end effector and add end effector mechanism in the urdf

File: src/inchworm/inchworm_description/urdf/inchworm.urdf.xacro (robot description, xacro)
@@ -58,9 +58,18 @@
             <inertia ixx="0.0" ixy="0.0" ixz="0.0" iyy="0.0" iyz="0.0" izz="0.0"/>
         </inertial>
+        <collision>
+            <origin xyz="0.0 0.0 -0.044" rpy="0.0 0.0 0.0"/>
+            <geometry>
+                <cylinder radius="0.0345" length="0.01"/>
+            </geometry>
+        </collision>
     </link>
     <link name="frontfoot_ee_link">
-        <inertial>
-            <origin xyz="0.0 0.0 0.0" rpy="0.0 0.0 0.0"/>
-            <mass value="0.1"/>
+        <gazebo>
+            <gravity>true</gravity>
+        </gazebo>
+        <inertial>
+            <origin xyz="0.0 0.0 0.0" rpy="0.0 0.0 0.0"/>
+            <mass value="10"/>
             <inertia ixx="0.0" ixy="0.0" ixz="0.0" iyy="0.0" iyz="0.0" izz="0.0"/>
         </inertial>
@@ -104,9 +113,18 @@
             <inertia ixx="0.0" ixy="0.0" ixz="0.0" iyy="0.0" iyz="0.0" izz="0.0"/>
         </inertial>
+        <collision>
+            <origin xyz="0.0 0.0 -0.044" rpy="0.0 0.0 0.0"/>
+            <geometry>
+                <cylinder radius="0.0345" length="0.01"/>
+            </geometry>
+        </collision>
     </link>
     <link name="backfoot_ee_link">
-        <inertial>
-            <origin xyz="0.0 0.0 0.0" rpy="0.0 0.0 0.0"/>
-            <mass value="0.1"/>
+        <gazebo>
+            <gravity>false</gravity>
+        </gazebo>
+        <inertial>
+            <origin xyz="0.0 0.0 0.0" rpy="0.0 0.0 0.0"/>
+            <mass value="10.0"/>
             <inertia ixx="0.0" ixy="0.0" ixz="0.0" iyy="0.0" iyz="0.0" izz="0.0"/>
         </inertial>

Commit message: Remove ee links because they cause issues

File: src/inchworm/inchworm_description/urdf/inchworm.urdf.xacro (robot description, xacro)
@@ -65,5 +65,5 @@
         </collision>
     </link>
-    <link name="frontfoot_ee_link">
+    <!-- <link name="frontfoot_ee_link">
         <gazebo>
             <gravity>true</gravity>
@@ -74,5 +74,5 @@
             <inertia ixx="0.0" ixy="0.0" ixz="0.0" iyy="0.0" iyz="0.0" izz="0.0"/>
         </inertial>
-    </link>
+    </link> -->
     <link name="c_link">
         <visual>
@@ -120,5 +120,5 @@
         </collision>
     </link>
-    <link name="backfoot_ee_link">
+    <!-- <link name="backfoot_ee_link">
         <gazebo>
             <gravity>false</gravity>
@@ -129,5 +129,5 @@
             <inertia ixx="0.0" ixy="0.0" ixz="0.0" iyy="0.0" iyz="0.0" izz="0.0"/>
         </inertial>
-    </link>
+    </link> -->
     <!-- Joint Transmission Macro -->
     <xacro:macro name="joint_transmission" params="prefix">
@@ -168,11 +168,9 @@
     </joint>
     <xacro:joint_transmission prefix="frontleg_frontfoot"/>
-    <joint name="frontfoot_ee_joint" type="fixed">
+    <!-- <joint name="frontfoot_ee_joint" type="fixed">
         <origin xyz="0.0 0.0 -0.0489" rpy="0.0 0.0 0.0"/>
         <parent link="frontfoot_link"/>
         <child link="frontfoot_ee_link"/>
-        <limit  effort="${joint_torque}"
-                velocity="${joint_speed * 2 * 3.14159 / 60 }"/>
-    </joint>
+    </joint> -->
     <joint name="main_c_joint" type="continuous">
         <origin xyz="0.0 0.0 0.0" rpy="-1.5707 1.5707 0"/>
@@ -202,10 +200,8 @@
     </joint>
     <xacro:joint_transmission prefix="backleg_backfoot"/>
-    <joint name="backfoot_ee_joint" type="fixed">
+    <!-- <joint name="backfoot_ee_joint" type="fixed">
         <origin xyz="0.0 0.0 -0.0489" rpy="0.0 0.0 0.0"/>
         <parent link="backfoot_link"/>
         <child link="backfoot_ee_link"/>
-        <limit  effort="${joint_torque}"
-                velocity="${joint_speed * 2 * 3.14159 / 60 }"/>
-    </joint>
+    </joint> -->
 </robot>

File: src/inchworm/inchworm_description/urdf/inchworm_static.urdf.xacro (robot description, xacro)
@@ -1,4 +1,4 @@
 <?xml version="1.0"?>
-<robot xmlns:xacro="http://wiki.ros.org/xacro" name="inchworm_static">
+<robot xmlns:xacro="http://wiki.ros.org/xacro" name="inchworm">
     <!-- Note: Only use this URDF when testing the inchworm kinematics.
     The inchworm will be fixed to a specific position as determined under 'Static Joint to World Frame' comment -->
@@ -70,12 +70,21 @@
             <inertia ixx="0.0" ixy="0.0" ixz="0.0" iyy="0.0" iyz="0.0" izz="0.0"/>
         </inertial>
-    </link>
-    <link name="frontfoot_ee_link">
-        <inertial>
-            <origin xyz="0.0 0.0 0.0" rpy="0.0 0.0 0.0"/>
-            <mass value="0.1"/>
-            <inertia ixx="0.0" ixy="0.0" ixz="0.0" iyy="0.0" iyz="0.0" izz="0.0"/>
-        </inertial>
-    </link>
+        <collision>
+            <origin xyz="0.0 0.0 -0.044" rpy="0.0 0.0 0.0"/>
+            <geometry>
+                <cylinder radius="0.0345" length="0.01"/>
+            </geometry>
+        </collision>
+    </link>
+    <!-- <link name="frontfoot_ee_link">
+        <gazebo>
+            <gravity>true</gravity>
+        </gazebo>
+        <inertial>
+            <origin xyz="0.0 0.0 0.0" rpy="0.0 0.0 0.0"/>
+            <mass value="10"/>
+            <inertia ixx="0.0" ixy="0.0" ixz="0.0" iyy="0.0" iyz="0.0" izz="0.0"/>
+        </inertial>
+    </link> -->
     <link name="c_link">
         <visual>
@@ -116,12 +125,21 @@
             <inertia ixx="0.0" ixy="0.0" ixz="0.0" iyy="0.0" iyz="0.0" izz="0.0"/>
         </inertial>
-    </link>
-    <link name="backfoot_ee_link">
-        <inertial>
-            <origin xyz="0.0 0.0 0.0" rpy="0.0 0.0 0.0"/>
-            <mass value="0.1"/>
-            <inertia ixx="0.0" ixy="0.0" ixz="0.0" iyy="0.0" iyz="0.0" izz="0.0"/>
-        </inertial>
-    </link>
+        <collision>
+            <origin xyz="0.0 0.0 -0.044" rpy="0.0 0.0 0.0"/>
+            <geometry>
+                <cylinder radius="0.0345" length="0.01"/>
+            </geometry>
+        </collision>
+    </link>
+    <!-- <link name="backfoot_ee_link">
+        <gazebo>
+            <gravity>false</gravity>
+        </gazebo>
+        <inertial>
+            <origin xyz="0.0 0.0 0.0" rpy="0.0 0.0 0.0"/>
+            <mass value="10.0"/>
+            <inertia ixx="0.0" ixy="0.0" ixz="0.0" iyy="0.0" iyz="0.0" izz="0.0"/>
+        </inertial>
+    </link> -->
     <!-- Joint Transmission Macro -->
     <xacro:macro name="joint_transmission" params="prefix">
@@ -162,5 +180,5 @@
     </joint>
     <xacro:joint_transmission prefix="frontleg_frontfoot"/>
-    <joint name="frontfoot_ee_joint" type="fixed">
+    <!-- <joint name="frontfoot_ee_joint" type="fixed">
         <origin xyz="0.0 0.0 -0.0489" rpy="0.0 0.0 0.0"/>
         <parent link="frontfoot_link"/>
@@ -168,5 +186,5 @@
         <limit  effort="${joint_torque}"
                 velocity="${joint_speed * 2 * 3.14159 / 60 }"/>
-    </joint>
+    </joint> -->
     <joint name="main_c_joint" type="continuous">
         <origin xyz="0.0 0.0 0.0" rpy="-1.5707 1.5707 0"/>
@@ -196,5 +214,5 @@
     </joint>
     <xacro:joint_transmission prefix="backleg_backfoot"/>
-    <joint name="backfoot_ee_joint" type="fixed">
+    <!-- <joint name="backfoot_ee_joint" type="fixed">
         <origin xyz="0.0 0.0 -0.0489" rpy="0.0 0.0 0.0"/>
         <parent link="backfoot_link"/>
@@ -202,4 +220,4 @@
         <limit  effort="${joint_torque}"
                 velocity="${joint_speed * 2 * 3.14159 / 60 }"/>
-    </joint>
+    </joint> -->
 </robot>
