Commit message: Add fkin but not tested

File: src/inchworm/inchworm_description/urdf/inchworm_base.urdf.xacro (robot description, xacro)
@@ -58,14 +58,6 @@
             </collision>
         </link>
-        <!-- <link name="frontfoot_ee_link">
-            <gazebo>
-                <gravity>true</gravity>
-            </gazebo>
-            <inertial>
-                <origin xyz="0.0 0.0 0.0" rpy="0.0 0.0 0.0"/>
-                <mass value="10"/>
-                <inertia ixx="0.0" ixy="0.0" ixz="0.0" iyy="0.0" iyz="0.0" izz="0.0"/>
-            </inertial>
-        </link> -->
+        <link name="frontfoot_ee_link">
+        </link>
         <link name="c_link">
             <visual>
@@ -113,14 +105,6 @@
             </collision>
         </link>
-        <!-- <link name="backfoot_ee_link">
-            <gazebo>
-                <gravity>false</gravity>
-            </gazebo>
-            <inertial>
-                <origin xyz="0.0 0.0 0.0" rpy="0.0 0.0 0.0"/>
-                <mass value="10.0"/>
-                <inertia ixx="0.0" ixy="0.0" ixz="0.0" iyy="0.0" iyz="0.0" izz="0.0"/>
-            </inertial>
-        </link> -->
+        <link name="backfoot_ee_link">
+        </link>
         <!-- Joint Transmission Macro -->
         <xacro:macro name="joint_transmission" params="prefix">
@@ -161,11 +145,9 @@
         </joint>
         <xacro:joint_transmission prefix="frontleg_frontfoot"/>
-        <!-- <joint name="frontfoot_ee_joint" type="fixed">
+        <joint name="frontfoot_ee_joint" type="fixed">
             <origin xyz="0.0 0.0 -0.0489" rpy="0.0 0.0 0.0"/>
             <parent link="frontfoot_link"/>
             <child link="frontfoot_ee_link"/>
-            <limit  effort="${joint_torque}"
-                    velocity="${joint_speed * 2 * 3.14159 / 60 }"/>
-        </joint> -->
+        </joint>
         <joint name="main_c_joint" type="continuous">
             <origin xyz="0.0 0.0 0.0" rpy="-1.5707 1.5707 0"/>
@@ -195,11 +177,9 @@
         </joint>
         <xacro:joint_transmission prefix="backleg_backfoot"/>
-        <!-- <joint name="backfoot_ee_joint" type="fixed">
+        <joint name="backfoot_ee_joint" type="fixed">
             <origin xyz="0.0 0.0 -0.0489" rpy="0.0 0.0 0.0"/>
             <parent link="backfoot_link"/>
             <child link="backfoot_ee_link"/>
-            <limit  effort="${joint_torque}"
-                    velocity="${joint_speed * 2 * 3.14159 / 60 }"/>
-        </joint> -->
+        </joint>
     </xacro:macro>
 </robot>

Commit message: Add joint command interface to the controller

File: src/inchworm/inchworm_description/urdf/inchworm_base.urdf.xacro (robot description, xacro)
@@ -58,6 +58,4 @@
             </collision>
         </link>
-        <link name="frontfoot_ee_link">
-        </link>
         <link name="c_link">
             <visual>
@@ -105,6 +103,8 @@
             </collision>
         </link>
-        <link name="backfoot_ee_link">
-        </link>
+        <!-- <link name="frontfoot_ee_link">
+        </link> -->
+        <!-- <link name="backfoot_ee_link">
+        </link> -->
         <!-- Joint Transmission Macro -->
         <xacro:macro name="joint_transmission" params="prefix">
@@ -145,9 +145,4 @@
         </joint>
         <xacro:joint_transmission prefix="frontleg_frontfoot"/>
-        <joint name="frontfoot_ee_joint" type="fixed">
-            <origin xyz="0.0 0.0 -0.0489" rpy="0.0 0.0 0.0"/>
-            <parent link="frontfoot_link"/>
-            <child link="frontfoot_ee_link"/>
-        </joint>
         <joint name="main_c_joint" type="continuous">
             <origin xyz="0.0 0.0 0.0" rpy="-1.5707 1.5707 0"/>
@@ -177,9 +172,14 @@
         </joint>
         <xacro:joint_transmission prefix="backleg_backfoot"/>
-        <joint name="backfoot_ee_joint" type="fixed">
+        <!-- <joint name="frontfoot_ee_joint" type="fixed">
+            <origin xyz="0.0 0.0 -0.0489" rpy="0.0 0.0 0.0"/>
+            <parent link="frontfoot_link"/>
+            <child link="frontfoot_ee_link"/>
+        </joint> -->
+        <!-- <joint name="backfoot_ee_joint" type="fixed">
             <origin xyz="0.0 0.0 -0.0489" rpy="0.0 0.0 0.0"/>
             <parent link="backfoot_link"/>
             <child link="backfoot_ee_link"/>
-        </joint>
+        </joint> -->
     </xacro:macro>
 </robot>

File: src/inchworm/inchworm_description/urdf/inchworm_static.urdf.xacro (robot description, xacro)
@@ -9,9 +9,4 @@
         </plugin>
     </gazebo>
-    <!-- Joint Properties -->
-    <xacro:property name="joint_speed" value="545"/>        <!-- in rpm -->
-    <xacro:property name="joint_torque" value="0.03525"/>   <!-- in N-m -->
-    <xacro:include filename="$(find inchworm_description)/urdf/inchworm_base.urdf.xacro"/>
-    <xacro:inchworm_base/>
     <!-- Static Joint to World Frame in Simulation -->
     <link name="world"/>
@@ -19,10 +14,7 @@
         <origin xyz="0.0 0.0 0.0" rpy="0.0 0.0 0.0"/>
         <parent link="world"/>
-        <!-- Uncomment below if you want to test general kinematics or end effector -->
         <child link="inchworm_main"/>
-        <!-- Uncomment below if you want to test front foot kinematics -->
-        <!-- <child link="backfoot_ee_link"/>  -->
-        <!-- Uncomment below if you want to test back foot kinematics -->
-        <!-- <child link="frontfoot_link"/>  -->
     </joint>
+    <xacro:include filename="$(find inchworm_description)/urdf/inchworm_base.urdf.xacro"/>
+    <xacro:inchworm_base/>
 </robot>

Commit message: Add better cmd_joint interface and add end effector cmd msg

File: src/inchworm/inchworm_description/urdf/inchworm_base.urdf.xacro (robot description, xacro)
@@ -3,6 +3,6 @@
     <xacro:macro name="inchworm_base">
         <!-- Joint Properties -->
-        <xacro:property name="joint_speed" value="545"/>        <!-- in rpm -->
-        <xacro:property name="joint_torque" value="0.03525"/>   <!-- in N-m -->
+        <xacro:property name="joint_speed" value="20"/>        <!-- in rpm -->
+        <xacro:property name="joint_torque" value="3.525"/>   <!-- in N-m -->
         <!-- Links -->
         <link name="inchworm_main">
@@ -48,5 +48,5 @@
             <inertial>
                 <origin xyz="0.0 0.0 0.0" rpy="0.0 0.0 0.0"/>
-                <mass value="0.09525"/>
+                <mass value="0.010"/>
                 <inertia ixx="358.56" ixy="0.0" ixz="0.0" iyy="337.47" iyz="0.0" izz="98.47"/>
             </inertial>
@@ -93,5 +93,5 @@
             <inertial>
                 <origin xyz="0.0 0.0 0.0" rpy="0.0 0.0 0.0"/>
-                <mass value="0.09525"/>
+                <mass value="10.0"/>
                 <inertia ixx="358.56" ixy="0.0" ixz="0.0" iyy="337.47" iyz="0.0" izz="98.47"/>
             </inertial>
@@ -103,8 +103,8 @@
             </collision>
         </link>
-        <!-- <link name="frontfoot_ee_link">
-        </link> -->
-        <!-- <link name="backfoot_ee_link">
-        </link> -->
+        <link name="frontfoot_ee_link">
+        </link>
+        <link name="backfoot_ee_link">
+        </link>
         <!-- Joint Transmission Macro -->
         <xacro:macro name="joint_transmission" params="prefix">
@@ -172,14 +172,14 @@
         </joint>
         <xacro:joint_transmission prefix="backleg_backfoot"/>
-        <!-- <joint name="frontfoot_ee_joint" type="fixed">
+        <joint name="frontfoot_ee_joint" type="fixed">
             <origin xyz="0.0 0.0 -0.0489" rpy="0.0 0.0 0.0"/>
             <parent link="frontfoot_link"/>
             <child link="frontfoot_ee_link"/>
-        </joint> -->
-        <!-- <joint name="backfoot_ee_joint" type="fixed">
+        </joint>
+        <joint name="backfoot_ee_joint" type="fixed">
             <origin xyz="0.0 0.0 -0.0489" rpy="0.0 0.0 0.0"/>
             <parent link="backfoot_link"/>
             <child link="backfoot_ee_link"/>
-        </joint> -->
+        </joint>
     </xacro:macro>
 </robot>
